Commit message: feat: integrated yolopv2 into the  planner

File: src/simulation_2025/urdf/camera.xacro (robot description, xacro)
@@ -25,7 +25,13 @@
         <origin xyz="1 0 0.8" rpy="0 0 0" />
     </joint>
+    <link name="camera_link_optical"></link>
+    <joint name="camera_optical_joint" type="fixed">
+        <origin xyz="0 0 0" rpy="${-pi/2} 0 ${-pi/2}"/>
+        <parent link="camera_link"/>
+        <child link="camera_link_optical"/>
+    </joint>
     <gazebo reference="camera_link">
         <sensor name="camera" type="camera">
-            <gz_frame_id>camera_link</gz_frame_id>
+            <gz_frame_id>camera_link_optical</gz_frame_id>
             <camera>
                 <horizontal_fov>1.91986</horizontal_fov>
@@ -38,9 +44,9 @@
                   <far>130</far>
                 </clip>
-              </camera>
-              <always_on>1</always_on>
-              <update_rate>100</update_rate>
-              <visualize>true</visualize>
-              <topic>camera</topic>
+            </camera>
+            <always_on>1</always_on>
+            <update_rate>100</update_rate>
+            <visualize>true</visualize>
+            <topic>camera</topic>
         </sensor>
     </gazebo>

File: src/simulation_2025/urdf/depth.xacro (robot description, xacro)
@@ -3,5 +3,5 @@
     <gazebo reference="camera_link">
         <sensor name="depth" type="depth_camera">
-            <gz_frame_id>camera_link</gz_frame_id>
+            <gz_frame_id>camera_link_optical</gz_frame_id>
             <camera>
                 <horizontal_fov>1.91986</horizontal_fov>
